File: hardware/ntp_tiny_matrix_clock.sch (KiCad schematic (older format))
At the start: 79 parts, among them J1 Barrel_Jack, J10 Conn_02x04_Odd_Even, J11 Conn_02x04_Odd_Even, J12 Conn_01x04_Male, J13 Conn_01x04_Male, J2 USB_B_Micro, J3 Conn_02x04_Odd_Even, J4 Conn_02x04_Odd_Even, J5 Conn_02x04_Odd_Even, J6 Conn_02x04_Odd_Even, J7 Conn_01x06_Male, J8 Conn_02x04_Odd_Even, J9 Conn_02x04_Odd_Even, Q1 Q_NPN_BEC, Q2 AO3401, Q3 AO3401, Q4 NJL7302L-F3, Q5 Q_NPN_BEC, Q6 Q_NPN_BEC, SW1 SW_PUSH_SMALL_H, U1 PCF8563, U2 NJW4132U2-C, U3 ESP32-WROOM, U4 W256064-XALG, U5 BME280, U7 JW5150A

Commit message: to use holtek led driver
Parts:
- added D8: LED_Small, LED_SMD:LED_0603_1608Metric, symbol Device:LED_Small
- added LED1: LED48x14, components:led_matrix_0402_48x14, symbol DeeComponents:LED48x14
- added R21: 4.7k, Resistor_SMD:R_0603_1608Metric, symbol ntp_tiny_matrix_clock-rescue:R-device-ntp_7seg_clock-rescue
- added U6, U8, U9: HT16D35A, Package_QFP:LQFP-48_7x7mm_P0.5mm, symbol DeeComponents:HT16D35A
- J10, J5: footprint Connector_PinHeader_1.27mm:PinHeader_2x04_P1.27mm_Vertical_SMD -> Connector_PinSocket_2.54mm:PinSocket_2x03_P2.54mm_Vertical_SMD; symbol ntp_tiny_matrix_clock-rescue:Conn_02x04_Odd_Even-Connector-ntp_7seg_clock-rescue -> Connector_Generic:Conn_02x03_Odd_Even
- J11, J6: footprint Connector_PinSocket_1.27mm:PinSocket_2x04_P1.27mm_Vertical_SMD -> Connector_PinSocket_2.54mm:PinSocket_2x03_P2.54mm_Vertical_SMD; symbol ntp_tiny_matrix_clock-rescue:Conn_02x04_Odd_Even-Connector-ntp_7seg_clock-rescue -> Connector_Generic:Conn_02x03_Odd_Even
- J3, J8: footprint Connector_PinHeader_1.27mm:PinHeader_2x04_P1.27mm_Vertical_SMD -> Connector_PinHeader_2.54mm:PinHeader_2x03_P2.54mm_Vertical_SMD; symbol ntp_tiny_matrix_clock-rescue:Conn_02x04_Odd_Even-Connector-ntp_7seg_clock-rescue -> Connector_Generic:Conn_02x03_Odd_Even
- J4, J9: footprint Connector_PinSocket_1.27mm:PinSocket_2x04_P1.27mm_Vertical_SMD -> Connector_PinHeader_2.54mm:PinHeader_2x03_P2.54mm_Vertical_SMD; symbol ntp_tiny_matrix_clock-rescue:Conn_02x04_Odd_Even-Connector-ntp_7seg_clock-rescue -> Connector_Generic:Conn_02x03_Odd_Even
Connections:
- net labels added: C0, C1, C10, C11, C12, C13, C14, C15, C16, C17, C18, C19, C2, C20, C21, C22, C23, C24, C25, C26, C27, C28, C29, C3, C30, C31, C32, C33, C34, C35, C36, C37, C38, C39, C4, C40, C41, C42, C43, C44, C45, C46, C47, C5, C6, C7, C8, C9, LED_RLAT, LED_SCK, LED_SIN, LED_SOUT, LED_~SLAT, R0, R1, R10, R11, R12, R13, R2, R3, R4, R5, R6, R7, R8, R9, STATUS
- wire segments 285 -> 294
Other:
- moved on the sheet: C10, C14, C15, C3, C9, D6, D7, Q1, Q5, Q6, R1, R14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

Commit message: LED matrix circuit trace design ongoing. Too much difficult.
Parts:
- added C22, C23, C24, C25, C26, C27: 1u/50V, Capacitor_SMD:C_0603_1608Metric, symbol Device:C
- added JP1, JP2: Jumper_NC_Small, components:J_0.25mm, symbol Device:Jumper_NC_Small
- added R22, R23, R24: 1k, Resistor_SMD:R_0603_1608Metric, symbol Device:R
- D5: footprint Diode_SMD:D_SOD-123 -> Diode_SMD:D_SOD-323
- J10, J11, J5, J6: footprint Connector_PinSocket_2.54mm:PinSocket_2x03_P2.54mm_Vertical_SMD -> Connector_PinSocket_1.27mm:PinSocket_2x04_P1.27mm_Vertical_SMD; symbol Connector_Generic:Conn_02x03_Odd_Even -> Connector_Generic:Conn_02x04_Odd_Even
- J3, J4, J8, J9: footprint Connector_PinHeader_2.54mm:PinHeader_2x03_P2.54mm_Vertical_SMD -> Connector_PinSocket_1.27mm:PinSocket_2x04_P1.27mm_Vertical_SMD; symbol Connector_Generic:Conn_02x03_Odd_Even -> Connector_Generic:Conn_02x04_Odd_Even
- LED1: footprint components:led_matrix_0402_48x14 -> thisproject:led_matrix_0402_48x14
Connections:
- net labels added: LD_OSC, LD_SYNC, LEDSPI_CS0, LEDSPI_CS1, LEDSPI_CS2, LEDVDD, LEDVSS, LED_VDD, LED_VSS, a0000, a0001, a0002, a0003, a0004, a0005, a0006, a0007, a0100, a0101, a0102, a0103, a0104, a0105, a0106, a0107, a0200, a0201, a0202, a0203, a0204, a0205, a0206, a0207, k0000, k0001, k0002, k0003, k0004, k0005, k0006, k0007, k0008, k0009, k0010, k0011, k0012, k0013, k0014, k0015, k0016, k0017, k0018, k0019, k0020, k0021, k0022, k0023, k0024, k0025, k0026, k0027, k0100, k0101, k0102, k0103, k0104, k0105, k0106, k0107, k0108, k0109, k0110, k0111, k0112, k0113, k0114, k0115, k0116, k0117, k0118, k0119, k0120, k0121, k0122, k0123, k0124, k0125, k0126, k0127, k0200, k0201, k0202, k0203, k0204, k0205, k0206, k0207, k0208, k0209, k0210, k0211, k0212, k0213, k0214, k0215, k0216, k0217, k0218, k0219, k0220, k0221, k0222, k0223, k0224, k0225, k0226, k0227
- net labels removed: C0, C1, C10, C11, C12, C13, C14, C15, C16, C17, C18, C19, C2, C20, C21, C22, C23, C24, C25, C26, C27, C28, C29, C3, C30, C31, C32, C33, C34, C35, C36, C37, C38, C39, C4, C40, C41, C42, C43, C44, C45, C46, C47, C5, C6, C7, C8, C9, R0, R1, R10, R11, R12, R13, R2, R3, R4, R5, R6, R7, R8, R9
- wire segments 294 -> 360
Other:
- note added: "Master"
- note added: "Slave"

Commit message: Almost all connection done; Traces are too narrow to keep signal integrity but there is no space left. sigh
Connections:
- wire segments 360 -> 367
Changed lines of the file:
@@
-$EndComp
-$Comp
-L Connector_Generic:Conn_02x04_Odd_Even J4
-U 1 1 5BF716ED
-P 1750 6300
-F 0 "J4" H 1800 6700 50  0000 C CNN
-F 1 "Conn_02x04_Odd_Even" H 1600 6550 50  0000 C CNN
-F 2 "Connector_PinSocket_1.27mm:PinSocket_2x04_P1.27mm_Vertical_SMD" H 1750 6300 50  0001 C CNN
-F 3 "~" H 1750 6300 50  0001 C CNN
-	1    1750 6300
-	1    0    0    1
 $EndComp
 $Comp
@@
 L power:+12V #PWR025
 U 1 1 5BFAE22D
-P 2150 6400
-F 0 "#PWR025" H 2150 6250 50  0001 C CNN
-F 1 "+12V" H 2165 6573 50  0000 C CNN
-F 2 "" H 2150 6400 50  0001 C CNN
-F 3 "" H 2150 6400 50  0001 C CNN
-	1    2150 6400
-	0    1    1    0
+P 2300 6250
+F 0 "#PWR025" H 2300 6100 50  0001 C CNN
+F 1 "+12V" H 2315 6423 50  0000 C CNN
+F 2 "" H 2300 6250 50  0001 C CNN
+F 3 "" H 2300 6250 50  0001 C CNN
+	1    2300 6250
+	0    1    -1   0
 $EndComp
 $Comp
@@
 L power:+3V3 #PWR040
 U 1 1 5C06C314
-P 2200 6100
-F 0 "#PWR040" H 2200 5950 50  0001 C CNN
-F 1 "+3V3" H 2215 6273 50  0000 C CNN
-F 2 "" H 2200 6100 50  0001 C CNN
-F 3 "" H 2200 6100 50  0001 C CNN
-	1    2200 6100
-	0    1    1    0
-$EndComp
-Wire Wire Line
-	2200 6100 2050 6100
+P 2200 6400
+F 0 "#PWR040" H 2200 6250 50  0001 C CNN
+F 1 "+3V3" H 2215 6573 50  0000 C CNN
+F 2 "" H 2200 6400 50  0001 C CNN
+F 3 "" H 2200 6400 50  0001 C CNN
+	1    2200 6400
+	0    1    -1   0
+$EndComp
+Wire Wire Line
+	2200 6400 2050 6400
 Connection ~ 2050 6100
-Connection ~ 2050 6200
 Text GLabel 1300 6950 0    60   Input ~ 0
 E_AIN
@@
 L power:GND #PWR047
 U 1 1 5C3EAA52
-P 2050 7300
-F 0 "#PWR047" H 2050 7050 50  0001 C CNN
-F 1 "GND" H 2055 7127 50  0000 C CNN
-F 2 "" H 2050 7300 50  0001 C CNN
-F 3 "" H 2050 7300 50  0001 C CNN
-	1    2050 7300
+P 2050 7250
+F 0 "#PWR047" H 2050 7000 50  0001 C CNN
+F 1 "GND" H 2055 7077 50  0000 C CNN
+F 2 "" H 2050 7250 50  0001 C CNN
+F 3 "" H 2050 7250 50  0001 C CNN
+	1    2050 7250
 	1    0    0    -1
 $EndComp
@@
 	0    1    1    0
 $EndComp
-Wire Wire Line
-	2150 6400 2050 6400
 Connection ~ 11600 1400
 Wire Wire Line
@@
 Wire Wire Line
 	1550 7200 850  7200
-Wire Wire Line
-	3350 7150 2650 7150
-Wire Wire Line
-	3350 7050 2650 7050
-Wire Wire Line
-	3350 6950 2650 6950
 Text Label 850  7200 0    50   ~ 0
 LCDSPI_CS
-Text Label 2650 7150 0    50   ~ 0
+Text Label 2550 6950 0    50   ~ 0
 LCDSPI_D~C
-Text Label 2650 6950 0    50   ~ 0
+Text Label 2550 7150 0    50   ~ 0
 LCDSPI_DAT
-Text Label 2650 7050 0    50   ~ 0
+Text Label 2550 7050 0    50   ~ 0
 LCDSPI_CLK
 $Comp
@@
 $EndComp
 Wire Wire Line
-	2050 6200 2050 6100
-Wire Wire Line
 	1550 6200 1550 6100
-Connection ~ 1550 6200
-Wire Wire Line
-	2050 6400 2050 6300
-Connection ~ 2050 6300
 Connection ~ 2050 7050
 Connection ~ 2050 7150
@@
 Text Label 13150 8200 1    31   ~ 0
 k0227
-Connection ~ 2050 6400
 Connection ~ 1550 6950
 Connection ~ 1550 7050
@@
 Connection ~ 3850 6100
 Connection ~ 3850 6400
-Connection ~ 3350 6950
-Connection ~ 3350 7050
-Connection ~ 3350 7150
 Connection ~ 3850 6950
 $Comp
@@
 Wire Wire Line
 	850  7350 850  7200
-Text Label 2650 7300 0    50   ~ 0
+Text Label 2500 7300 0    50   ~ 0
 LEDSPI_CS2
-Wire Wire Line
-	2650 7300 2650 7150
 Wire Wire Line
 	2250 9200 2250 9900
@@
 Wire Wire Line
 	1550 6400 1550 6300
-Connection ~ 1550 6400
 Wire Wire Line
 	1550 7250 1550 7450
@@
 Text Label 15500 1500 0    50   ~ 0
 LEDVDD
+Wire Wire Line
+	2500 6950 2500 7300
+Wire Wire Line
+	2500 6950 3350 6950
+Connection ~ 3350 6950
+Wire Wire Line
+	2550 7050 3350 7050
+Connection ~ 3350 7050
+Wire Wire Line
+	2550 7150 3350 7150
+Connection ~ 3350 7150
+Connection ~ 1550 6200
+Connection ~ 1550 6400
+$Comp
+L Connector_Generic:Conn_02x04_Odd_Even J4
+U 1 1 5BF716ED
+P 1750 6300
+F 0 "J4" H 1800 6700 50  0000 C CNN
+F 1 "Conn_02x04_Odd_Even" H 1600 6550 50  0000 C CNN
+F 2 "Connector_PinSocket_1.27mm:PinSocket_2x04_P1.27mm_Vertical_SMD" H 1750 6300 50  0001 C CNN
+F 3 "~" H 1750 6300 50  0001 C CNN
+	1    1750 6300
+	1    0    0    1
+$EndComp
+Wire Wire Line
+	2300 6250 2250 6250
+Wire Wire Line
+	2250 6250 2250 6300
+Wire Wire Line
+	2250 6300 2050 6300
+Connection ~ 2050 6200
+Text Label 2200 6050 0    50   ~ 0
+LED_VSS
+Text Label 2200 5950 0    50   ~ 0
+LED_VDD
+Wire Wire Line
+	2200 6050 2150 6050
+Wire Wire Line
+	2150 6050 2150 6200
+Wire Wire Line
+	2150 6200 2050 6200
+Connection ~ 2050 6300
+Wire Wire Line
+	2050 6100 2100 6100
+Wire Wire Line
+	2100 6100 2100 5950
+Wire Wire Line
+	2100 5950 2200 5950
+Connection ~ 2050 6400
+Wire Wire Line
+	3850 6850 3850 6950
+Connection ~ 3850 6850
 $EndSCHEMATC

Commit message: Routing ongoing...
Connections:
- wire segments 367 -> 363
Changed lines of the file:
@@
 	2200 6400 2050 6400
 Connection ~ 2050 6100
-Text GLabel 1300 6950 0    60   Input ~ 0
+Text GLabel 1350 7250 0    60   Input ~ 0
 E_AIN
-Text GLabel 1300 7050 0    60   Input ~ 0
+Text GLabel 3950 6100 2    60   Input ~ 0
 E_BUTTON
 Wire Wire Line
 	1550 6950 1300 6950
-Wire Wire Line
-	1300 7050 1550 7050
 Text Label 5450 1100 0    50   ~ 0
 VIN
@@
 	15250 6750 14500 6750
 Wire Wire Line
-	1550 7200 850  7200
-Text Label 850  7200 0    50   ~ 0
+	3850 7150 4550 7150
+Text Label 4550 7150 2    50   ~ 0
 LCDSPI_CS
 Text Label 2550 6950 0    50   ~ 0
@@
 Wire Wire Line
 	3850 6400 3850 6300
-Connection ~ 3850 6200
-Wire Wire Line
-	3850 6200 3850 6100
 Connection ~ 3850 6300
-Wire Wire Line
-	3850 6300 3850 6200
 $Comp
 L power:GND #PWR0108
 U 1 1 5C12F68B
-P 3850 7250
-F 0 "#PWR0108" H 3850 7000 50  0001 C CNN
-F 1 "GND" H 3855 7077 50  0000 C CNN
-F 2 "" H 3850 7250 50  0001 C CNN
-F 3 "" H 3850 7250 50  0001 C CNN
-	1    3850 7250
-	1    0    0    -1
+P 3850 6850
+F 0 "#PWR0108" H 3850 6600 50  0001 C CNN
+F 1 "GND" H 3855 6677 50  0000 C CNN
+F 2 "" H 3850 6850 50  0001 C CNN
+F 3 "" H 3850 6850 50  0001 C CNN
+	1    3850 6850
+	0    -1   -1   0
 $EndComp
 Wire Wire Line
@@
 Connection ~ 2050 7050
 Connection ~ 2050 7150
-Wire Wire Line
-	3850 7250 3850 7150
 Connection ~ 3850 7050
 Wire Wire Line
 	3850 7050 3850 6950
 Connection ~ 3850 7150
-Wire Wire Line
-	3850 7150 3850 7050
 Wire Wire Line
 	2050 7050 2050 6950
@@
 Wire Wire Line
 	2050 7150 2050 7250
-Wire Wire Line
-	1550 7200 1550 7150
 $Comp
 L DeeComponents:LED48x14 LED1
@@
 Wire Wire Line
 	5250 4700 5050 4700
-Text GLabel 1400 7450 0    50   Input ~ 0
+Text GLabel 3950 6200 2    50   Input ~ 0
 STATUS
 Wire Wire Line
@@
 k0227
 Connection ~ 1550 6950
-Connection ~ 1550 7050
-Connection ~ 1550 7150
 Connection ~ 2050 6950
 Connection ~ 2050 7250
@@
 Connection ~ 3350 6200
 Connection ~ 3350 6400
-Connection ~ 3850 6100
 Connection ~ 3850 6400
 Connection ~ 3850 6950
@@
 LEDSPI_CS0
 Connection ~ 3350 6850
-Text Label 850  7350 0    50   ~ 0
+Text Label 4550 7000 2    50   ~ 0
 LEDSPI_CS1
 Wire Wire Line
-	850  7350 850  7200
+	4550 7000 4550 7150
 Text Label 2500 7300 0    50   ~ 0
 LEDSPI_CS2
@@
 	1550 6400 1550 6300
 Wire Wire Line
-	1550 7250 1550 7450
-Wire Wire Line
-	1550 7450 1400 7450
-Connection ~ 1550 7250
-Wire Wire Line
 	3350 6200 3350 6100
-Wire Wire Line
-	3350 6100 2650 6100
-Text Label 2650 6100 0    50   ~ 0
-LEDVSS
-Wire Wire Line
-	3350 6300 2650 6300
-Text Label 2650 6300 0    50   ~ 0
-LEDVDD
 $Comp
 L Device:Jumper_NC_Small JP1
@@
 	3850 6850 3850 6950
 Connection ~ 3850 6850
+Wire Wire Line
+	3950 6100 3850 6100
+Connection ~ 3850 6100
+Wire Wire Line
+	3950 6200 3850 6200
+Connection ~ 3850 6200
+Wire Wire Line
+	1550 7050 1550 7150
+Connection ~ 1550 7050
+Connection ~ 1550 7150
+$Comp
+L power:GND #PWR054
+U 1 1 5C31DCEF
+P 1300 6950
+F 0 "#PWR054" H 1300 6700 50  0001 C CNN
+F 1 "GND" H 1305 6777 50  0000 C CNN
+F 2 "" H 1300 6950 50  0001 C CNN
+F 3 "" H 1300 6950 50  0001 C CNN
+	1    1300 6950
+	1    0    0    -1
+$EndComp
+$Comp
+L power:GND #PWR?
+U 1 1 5C31FBF2
+P 3350 6400
+F 0 "#PWR?" H 3350 6150 50  0001 C CNN
+F 1 "GND" H 3355 6227 50  0000 C CNN
+F 2 "" H 3350 6400 50  0001 C CNN
+F 3 "" H 3350 6400 50  0001 C CNN
+	1    3350 6400
+	1    0    0    -1
+$EndComp
+Wire Wire Line
+	3350 6300 3350 6200
+Wire Wire Line
+	1550 7050 1550 6950
+Wire Wire Line
+	1550 7250 1350 7250
+Connection ~ 1550 7250
 $EndSCHEMATC
